File: ESP32_S3_MCU.kicad_sch (KiCad schematic)
At the start: 14 parts, among them SW2 SW_Push, SW4 SW_Push, U4 ESP32-S3-WROOM-1, X3 32.768KHz

Commit message: pcb updates & improvements
Parts:
- removed C16: 100n, Capacitor_SMD:C_0402_1005Metric, symbol Device:C_Small
- removed C55, C56: 12p, Capacitor_SMD:C_0402_1005Metric, symbol Device:C_Small
- removed R10, R8: 5k1, Resistor_SMD:R_0603_1608Metric, symbol Device:R_Small
- removed X3: 32.768KHz, Crystal:Crystal_SMD_3225-4Pin_3.2x2.5mm, symbol Device:Crystal_GND24_Small
- C19: value 100n -> 1uf
- R12: value 5k1 -> 10k
- SW2: value SW_Push -> RESET
- SW4: value SW_Push -> BOOT
Connections:
- net +3V3: now also R12.2; no longer R12.1
- net ENABLE: now also C15.1, R12.1, SW2.2; no longer R12.2
- net XTAL_N: no longer names the net of U4.9 (IO16)
- net XTAL_P: no longer names the net of U4.8 (IO15)
Other:
- moved on the sheet: C10, C15, C19, C9, R12, SW2, SW4, U4
