File: connectors.kicad_sch (KiCad schematic)
At the start: 20 parts, among them J1 USB_C_Receptacle_USB2.0, J10 JTAG, J11 UART, J2 Power_Input, J3 Conn_01x11_Socket, J4 MOTOR_1_OUTPUT, J5 MOTOR_2_OUTPUT, J6 MOTOR_3_OUTPUT, J7 MOTOR_4_OUTPUT, J8 Conn_01x03_Socket, J9 Conn_01x11_Socket, U3 USBLC6-2SC6

Commit message: pcb updates & improvements
Parts:
- removed JP1: Jumper_PMODE, Connector_PinHeader_2.54mm:PinHeader_1x03_P2.54mm_Vertical_SMD_Pin1Right, symbol Jumper:Jumper_3_Bridged12
- added JP2: MOTOR_PMODE, Jumper:SolderJumper-3_P2.0mm_Open_TrianglePad1.0x1.5mm, symbol Jumper:SolderJumper_3_Open
- J1: value USB_C_Receptacle_USB2.0 -> USB-C
- J8: value Conn_01x03_Socket -> PWR
Connections:
- net +3V3: now also JP2.1 (A)
- net GND: now also JP2.3 (B)
- net MOTOR_PMODE: now also JP2.2 (C)
Other:
- moved on the sheet: D4, H1, H2, H3, H4, J1, J10, J3, J9, R2, R3, U3
